File: MG.brd (EAGLE design)
At the start: 62.2 x 24.3 mm, 42 parts, among them IC1 LM4871MM_NOPB, J1 BWIPX-1-001E, Q1 S9013, Q2 S9013, X1 BM04B-SRSS-TB, X2 BM04B-SRSS-TB, X3 BM04B-SRSS-TB

Commit message: second
Routing:
- net VDD_3.3V: track 112.7 -> 117.4 mm
Changed lines of the file:
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@@
 <drawing>
 <settings>
-<setting alwaysvectorfont="yes"/>
+<setting alwaysvectorfont="no"/>
 <setting verticaltext="up"/>
 </settings>
@@
 <via x="-24.627" y="19.669" extent="1-16" drill="0.2"/>
 <wire x1="-31.219" y1="9.086" x2="-36.627" y2="14.494" width="0.3048" layer="1"/>
+<wire x1="-50.202" y1="19.669" x2="-52.213" y2="19.669" width="0.1524" layer="1"/>
+<wire x1="-52.213" y1="19.669" x2="-54.102" y2="17.78" width="0.1524" layer="1"/>
 </signal>
 <signal name="VDD_AV_3.3V">
